File: Hardware/rev1/Interface_and_debugging.kicad_sch (KiCad schematic)
At the start: 8 parts, among them J1 USB_C_Receptacle_USB2.0_14P, J2 Conn_ARM_JTAG_SWD_10, Y1 16MHz

Commit message: UUUUHHH
Parts:
- removed C12, C13: 10p, Capacitor_SMD:C_0402_1005Metric, symbol Device:C
- removed Y1: 16MHz, Crystal:Crystal_SMD_3225-4Pin_3.2x2.5mm, symbol Device:Crystal_GND23_Small
- added U4: W25Q128JVS, Package_SO:SOIC-8_5.23x5.23mm_P1.27mm, symbol Memory_Flash:W25Q128JVS
Connections:
- net +3.3V: now also U4.8 (VCC)
- net GND: now also U4.4 (GND)
- new net Flash Data In: U4.5 (DI(IO0))
- new net Flash Data Out: U4.2 (DO(IO1))
- new net SPI_CLK: U4.6 (CLK)
- no-connect marks 0 -> 3
Other:
- note removed: "CL=2*(CLO-Cs) = 2*(10-5) = 10pF"
- moved on the sheet: J1, R1, R2, R4
